File: MCU Datalogger.kicad_sch (KiCad schematic)
At the start: 25 parts, among them U1 24LC1025, U2 DS1337S+, U3 24LC1025, U4 ATMEGA328P-AU, Y1 32.768 KHz, Y2 16MHz

Commit message: trying to merge master in to get the same vcc net
Connections:
- net Vcc: no longer BT1.1 (+), C5.1, D2.2 (A), U4.18 (AVCC), U4.4 (VCC)
- new net: BT1.1 (+), C5.1, D2.2 (A), U4.18 (AVCC), U4.4 (VCC)
Changed lines of the file:
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@@
-    (effects (font (size 1.27 1.27)) (justify left bottom))
-  )
-  (label "Vcc" (at 253.365 36.195 0)
     (effects (font (size 1.27 1.27)) (justify left bottom))
   )
@@
     (effects (font (size 1.27 1.27)) (justify left bottom))
   )
-  (label "Vcc" (at 255.27 36.195 0)
-    (effects (font (size 1.27 1.27)) (justify left bottom))
-  )

Commit message: finished upsizing the vcc tracks that didn't update automatically after I added the vcc net going into the battery
Connections:
- net Vcc: now also BT1.1 (+), C5.1, D2.2 (A), U4.18 (AVCC), U4.4 (VCC)
Changed lines of the file:
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@@
     (effects (font (size 1.27 1.27)) (justify right bottom))
+  )
+  (label "Vcc" (at 253.365 36.195 0)
+    (effects (font (size 1.27 1.27)) (justify left bottom))
   )
   (label "Vcc" (at 182.88 135.89 180)
